Commit message: Correct wheels

File: description/diffbot_description.xacro (robot description, xacro)
@@ -1,16 +1,15 @@
 <?xml version="1.0"?>
 <robot xmlns:xacro="http://www.ros.org/wiki/xacro">
-  <xacro:macro name="diffbot" params="prefix">
     <!-- Constants for robot dimensions -->
     <xacro:property name="PI" value="3.1415926535897931"/>
-    <xacro:property name="base_mass" value="12.0" /> <!-- arbitrary value for base mass -->
+    <xacro:property name="base_mass" value="12.0" /> <!-- value for base mass -->
     <xacro:property name="base_width" value="0.6" /> <!--size in X -->
     <xacro:property name="base_length" value="0.3" /> <!--size in Y -->
     <xacro:property name="base_height" value="0.2" />
     <xacro:property name="wheelbase" value="0.375" />
-    <xacro:property name="wheel_mass" value="1.0" /> <!-- arbitrary value for wheel mass -->
+    <xacro:property name="wheel_mass" value="1.0" /> <!-- wheel mass -->
     <xacro:property name="wheel_len" value="0.065" />
     <xacro:property name="wheel_radius" value="0.14" />
-    <xacro:property name="caster_wheel_mass" value="0.1" /> <!-- arbitrary value for caster wheel mass -->
+    <xacro:property name="caster_wheel_mass" value="0.1" /> <!-- value for caster wheel mass -->
     <xacro:property name="caster_wheel_radius" value="0.08" />
     <xacro:property name="z_offset" value="-${base_height/2}" /> <!-- Space btw top of beam and the each joint -->
@@ -19,10 +18,11 @@
     <link name="base_link">
     </link>
-    <joint name="${prefix}chassis_joint" type="fixed">
+    <!-- Chassis Link -->
+    <joint name="chassis_joint" type="fixed">
       <parent link="base_link"/>
-      <child link="${prefix}chassis_link"/>
+      <child link="chassis"/>
       <origin xyz="${x_body_offset} 0.0 ${base_height/2}"/>
     </joint>
-    <link name="${prefix}chassis_link">
+    <link name="chassis">
       <collision>
         <origin xyz="0 0 0" rpy="0 0 0"/>
@@ -45,46 +45,52 @@
           iyy="${base_mass / 12.0 * (base_height*base_height + base_width*base_width)}" iyz="0.0"
           izz="${base_mass / 12.0 * (base_width*base_width + base_length*base_length)}"/>
+      </inertial>
+    </link>
+    <gazebo reference="chassis">
+      <material>Gazebo/Orange</material>
+    </gazebo>
+    <!-- left wheel Link -->
+    <joint name="left_wheel_joint" type="continuous">
+      <parent link="base_link"/>
+      <child link="left_wheel"/>
+      <origin xyz="0.0 ${wheelbase/2} 0.0" rpy="${PI/2} 0 0"/>
+      <axis xyz="0 0 -1"/>
+      <dynamics damping="0.2"/>
+    </joint>
+    <link name="left_wheel">
+      <collision>
+        <origin xyz="0 0 0" rpy="0 0 0"/>
+        <geometry>
+          <cylinder length="${wheel_len}" radius="${wheel_radius}"/>
+        </geometry>
+      </collision>
+      <visual>
+        <origin xyz="0 0 0" rpy="0 0 0"/>
+        <geometry>
+          <cylinder length="${wheel_len}" radius="${wheel_radius}"/>
+        </geometry>
+        <material name="black"/>
+      </visual>
+      <inertial>
+        <origin xyz="0 0 0" rpy="0 0 0"/>
+        <mass value="${wheel_mass}"/>
+        <inertia
+          ixx="${wheel_mass / 12.0 * (3*wheel_radius*wheel_radius + wheel_len*wheel_len)}" ixy="0.0" ixz="0.0"
+          iyy="${wheel_mass / 12.0 * (3*wheel_radius*wheel_radius + wheel_len*wheel_len)}" iyz="0.0"
+          izz="${wheel_mass / 2.0 * wheel_radius*wheel_radius}"/>
         </inertial>
       </link>
-      <joint name="${prefix}left_wheel_joint" type="continuous">
+        <gazebo reference="left_wheel">
+          <material>Gazebo/Black</material>
+        </gazebo>
+      <joint name="right_wheel_joint" type="continuous">
         <parent link="base_link"/>
-        <child link="${prefix}left_wheel"/>
-        <origin xyz="0.0 ${wheelbase/2} 0.0" rpy="${PI/2} 0 0"/>
-        <axis xyz="0 0 1"/>
-        <dynamics damping="0.2"/>
-      </joint>
-      <!-- left wheel Link -->
-      <link name="${prefix}left_wheel">
-        <collision>
-          <origin xyz="0 0 0" rpy="$0 0 0"/>
-          <geometry>
-            <cylinder length="${wheel_len}" radius="${wheel_radius}"/>
-          </geometry>
-        </collision>
-        <visual>
-          <origin xyz="0 0 0" rpy="0 0 0"/>
-          <geometry>
-            <cylinder length="${wheel_len}" radius="${wheel_radius}"/>
-          </geometry>
-          <material name="black"/>
-        </visual>
-        <inertial>
-          <origin xyz="0 0 0" rpy="0 0 0"/>
-          <mass value="${wheel_mass}"/>
-          <inertia
-            ixx="${wheel_mass / 12.0 * (3*wheel_radius*wheel_radius + wheel_len*wheel_len)}" ixy="0.0" ixz="0.0"
-            iyy="${wheel_mass / 12.0 * (3*wheel_radius*wheel_radius + wheel_len*wheel_len)}" iyz="0.0"
-            izz="${wheel_mass / 2.0 * wheel_radius*wheel_radius}"/>
-          </inertial>
-        </link>
-      <joint name="${prefix}right_wheel_joint" type="continuous">
-        <parent link="base_link"/>
-        <child link="${prefix}right_wheel"/>
+        <child link="right_wheel"/>
         <origin xyz="0.0 -${wheelbase/2} 0.0" rpy="${PI/2} 0 0"/>
-        <axis xyz="0 0 1"/>
+        <axis xyz="0 0 -1"/>
         <dynamics damping="0.2"/>
       </joint>
       <!-- right wheel Link -->
-      <link name="${prefix}right_wheel">
+      <link name="right_wheel">
         <collision>
           <origin xyz="0 0 0" rpy="0 0 0"/>
@@ -109,11 +115,14 @@
           </inertial>
         </link>
-      <joint name="${prefix}caster_frontal_wheel_joint" type="fixed">
+        <gazebo reference="right_wheel">
+          <material>Gazebo/Black</material>
+        </gazebo>
+      <joint name="caster_frontal_wheel_joint" type="fixed">
         <parent link="base_link"/>
-        <child link="${prefix}caster_frontal_wheel"/>
+        <child link="caster_frontal_wheel"/>
         <origin xyz="${x_body_offset * 2} 0 ${caster_wheel_radius - wheel_radius}" rpy="0 0 0"/>
       </joint>
       <!-- caster front wheel Link -->
-      <link name="${prefix}caster_frontal_wheel">
+      <link name="caster_frontal_wheel">
         <collision>
           <origin xyz="0 0 0" rpy="0 0 0"/>
@@ -138,4 +147,8 @@
           </inertial>
         </link>
-  </xacro:macro>
+        <gazebo reference="caster_frontal_wheel">
+          <material>Gazebo/White</material>
+          <mu1 value="0.001"/>
+          <mu2 value="0.001"/>
+        </gazebo>
 </robot>

File: description/robot.urdf.xacro (robot description, xacro)
@@ -2,8 +2,9 @@
 <robot xmlns:xacro="http://www.ros.org/wiki/xacro"  name="robot">
     <xacro:arg name="prefix" default="" />
-    <xacro:include filename="diffbot_description.urdf.xacro" />
+    <xacro:include filename="diffbot_description.xacro" />
+    <xacro:include filename="gazebo_control.xacro" />
     <!-- Import Rviz colors -->
     <xacro:include filename="diffbot.materials.xacro" />
     <!-- to make Prefixes work -->
-    <xacro:diffbot prefix="$(arg prefix)" />
+    <!-- <xacro:diffbot prefix="$(arg prefix)" /> -->
 </robot>

Commit message: Gazebo Working

File: description/diffbot_description.xacro (robot description, xacro)
@@ -62,5 +62,5 @@
         <origin xyz="0 0 0" rpy="0 0 0"/>
         <geometry>
-          <cylinder length="${wheel_len}" radius="${wheel_radius}"/>
+          <sphere radius="${wheel_radius}"/>
         </geometry>
       </collision>
@@ -96,5 +96,5 @@
           <origin xyz="0 0 0" rpy="0 0 0"/>
           <geometry>
-            <cylinder length="${wheel_len}" radius="${wheel_radius}"/>
+            <sphere radius="${wheel_radius}"/>
           </geometry>
         </collision>

File: description/robot.urdf.xacro (robot description, xacro)
@@ -3,5 +3,6 @@
     <xacro:arg name="prefix" default="" />
     <xacro:include filename="diffbot_description.xacro" />
-    <xacro:include filename="gazebo_control.xacro" />
+    <!-- <xacro:include filename="gazebo_control.xacro" /> -->
+    <xacro:include filename="ros2_control.xacro" />
     <!-- Import Rviz colors -->
     <xacro:include filename="diffbot.materials.xacro" />
