Commit message: It lives

File: description/ros2_control.xacro (robot description, xacro)
@@ -5,4 +5,12 @@
             <plugin>hover_diffdrive/HoverDiffDrive</plugin>
         </hardware>
+        <joint name="right_wheel_joint">
+            <command_interface name="velocity">
+                <param name="min">-10</param>
+                <param name="max">10</param>
+            </command_interface>
+            <state_interface name="position"/>
+            <state_interface name="velocity"/>
+        </joint>
         <joint name="left_wheel_joint">
             <command_interface name="velocity">
@@ -10,14 +18,6 @@
                 <param name="max">10</param>
             </command_interface>
+            <state_interface name="position"/>
             <state_interface name="velocity"/>
-            <state_interface name="position"/>
-        </joint>
-        <joint name="right_wheel_joint">
-            <command_interface name="velocity">
-                <param name="min">-10</param>
-                <param name="max">10</param>
-            </command_interface>
-            <state_interface name="velocity"/>
-            <state_interface name="position"/>
         </joint>
     </ros2_control>
